File: KiCad/Tesla-ADM2001.kicad_sch (KiCad schematic)
At the start: 35 parts, among them U1 DE113-RS-20/7.5

Commit message: Update Tesla-ADM2001.kicad_sch
Parts:
- removed R14: R, symbol Device:R
- added R14: 1MΩ, symbol Device:R_Potentiometer_Trim
Connections:
- net LO_BAT is gone; now on net LO BAT: U1.38 (LO_BAT)
- net SE is gone; now on net SENSE: DD1.21 (BP/GND)
- net GND: now also DD2.7 (Vss), DD2.7 (Vss), DD2.7 (Vss), DD2.7 (Vss)
- net U+: now also DD2.14 (Vdd), DD2.14 (Vdd), R8.1, R14.1; no longer BT1.1 (+), DD1.1 (V+), R2.2, VD3.1 (K)
- net U_{SS}: now also BT1.1 (+), DD1.1 (V+), R2.2, VD3.1 (K), VT1.2 (B)
- net at VT1.1 (C): now also DD2.8, R8.2
- net at R7.1, VT1.3 (E): now also R14.2, R14.3
- net D: now reaches DD2.11
- net SENSE: now reaches DD2.12, DD2.9, R10.2, R11.2, R12.2, R13.2
- net AB4: now reaches DD1.19 (AB4)
- net AB4: now also U1.3 (K)
- net POL: now reaches DD1.20 (POL)
- net POL: now also U1.2 (-)
- net AC: now reaches R13.1
- net LO BAT: now reaches DD2.10
- net 1A renamed A1
- net 1B renamed B1
- net 1C renamed C1
- net 1D renamed D1
- net 1E renamed E1
- net 1F renamed F1
- net 1G renamed G1
- net 2A renamed A2
- net 2B renamed B2
- net 2C renamed C2
- net 2D renamed D2
- net D2: now also DD1.14 (E2)
- net 2E renamed E2
- net E2: no longer DD1.14 (E2)
- net 2F renamed F2
- net 2G renamed G2
- net 3A renamed A3
- net 3B renamed B3
- net 3C renamed C3
- net 3D renamed D3
- net 3E renamed E3
- net 3F renamed F3
- net 3G renamed G3
Other:
- moved on the sheet: DD2B, DD2D, R7, R8, VT1
